Commit message: working on g1 - whole body

File: description_files/urdf/g1_29dof.urdf (robot description, URDF)
Before this commit: robot g1_29dof_rev_1_0, 57 links, 56 joints
Joints:
- joint left_knee_joint: limit lower=-0.087267 upper=2.8798 effort=139 velocity=20 -> lower=0.0 upper=2.1 effort=139 velocity=20
- joint right_knee_joint: limit lower=-0.087267 upper=2.8798 effort=139 velocity=20 -> lower=0.0 upper=2.1 effort=139 velocity=20
- joint waist_pitch_joint: limit lower=-0.52 upper=0.52 effort=50 velocity=37 -> lower=-0.42 upper=0.42 effort=50 velocity=37
- joint waist_roll_joint: limit lower=-0.52 upper=0.52 effort=50 velocity=37 -> lower=-0.42 upper=0.42 effort=50 velocity=37
- joint waist_yaw_joint: limit lower=-2.618 upper=2.618 effort=88 velocity=32 -> lower=-1.5 upper=1.5 effort=88 velocity=32
